Commit message: Update src packages

File: src/ rospital_description/urdf/imu.xacro (robot description, xacro)
@@ -5,14 +5,14 @@
     <inertial>
       <origin
-        xyz="-0.000320929221288936 -0.000281016175887928 0.000656651591240558"
+        xyz="0.000281016175887924 -0.000320929221288936 0.000656651591240559"
         rpy="0 0 0" />
       <mass
         value="0.000491630657107432" />
       <inertia
-        ixx="2.60740156632658E-08"
-        ixy="1.20559518329717E-10"
-        ixz="1.03040853232499E-10"
-        iyy="1.05219690062939E-08"
-        iyz="8.68518895699746E-11"
+        ixx="1.05219690062939E-08"
+        ixy="-1.20559518329718E-10"
+        ixz="-8.68518895699743E-11"
+        iyy="2.60740156632658E-08"
+        iyz="1.03040853232499E-10"
         izz="3.63603146259296E-08" />
     </inertial>
@@ -23,5 +23,5 @@
       <geometry>
         <mesh
-          filename="package://rospital_description/meshes/IMU_Link.STL" />
+          filename="package://rospital_description/meshes/IMU_link.STL" />
       </geometry>
       <material
@@ -37,5 +37,5 @@
       <geometry>
         <mesh
-          filename="package://rospital_description/meshes/IMU_Link.STL" />
+          filename="package://rospital_description/meshes/IMU_link.STL" />
       </geometry>
     </collision>
@@ -45,5 +45,5 @@
     type="fixed">
     <origin
-      xyz="-0.016497 0.002 0.032"
+      xyz="0 0 0.005"
       rpy="0 0 0" />
     <parent

File: src/ rospital_description/urdf/lidar.xacro (robot description, xacro)
@@ -5,15 +5,15 @@
     <inertial>
       <origin
-        xyz="0.0067665301166636 -9.19261110874925E-05 -0.00738187226715975"
+        xyz="-4.16811316961141E-07 -0.00020012090060817 0.0126456553172981"
         rpy="0 0 0" />
       <mass
-        value="1.33076913637071" />
+        value="0.00949435768129115" />
       <inertia
-        ixx="0.00061491794045409"
-        ixy="-8.01984318977561E-07"
-        ixz="0.00015824302591117"
-        iyy="0.000960697335617222"
-        iyz="-3.09162986587468E-06"
-        izz="0.00109815200027136" />
+        ixx="3.81407368895801E-06"
+        ixy="-2.89093384914113E-11"
+        ixz="2.07953967746501E-11"
+        iyy="3.81525913149567E-06"
+        iyz="-8.08800420939772E-10"
+        izz="4.9344522853465E-06" />
     </inertial>
     <visual>
@@ -23,10 +23,10 @@
       <geometry>
         <mesh
-          filename="package://rospital_description/meshes/Lidar_Link.STL" />
+          filename="package://rospital_description/meshes/laser_link.STL" />
       </geometry>
       <material
         name="">
         <color
-          rgba="0.792156862745098 0.819607843137255 0.933333333333333 1" />
+          rgba="0.0823529411764706 0.0823529411764706 0.0823529411764706 1" />
       </material>
     </visual>
@@ -37,5 +37,5 @@
       <geometry>
         <mesh
-          filename="package://rospital_description/meshes/Lidar_Link.STL" />
+          filename="package://rospital_description/meshes/laser_link.STL" />
       </geometry>
     </collision>
@@ -45,5 +45,5 @@
     type="fixed">
     <origin
-      xyz="0.015374 0.00030891 0.16515"
+      xyz="0.197743015846854 0.0027430158468545 0.159099867903085"
       rpy="0 0 0" />
     <parent

File: src/ rospital_description/urdf/rospital_core.xacro (robot description, xacro)
@@ -1,3 +1,3 @@
-<?xml version="1.0"?>
+<?xml version="1.0" ?>
 <robot xmlns:xacro="http://ros.org/wiki/xacro">
   <link name="base_footprint"/>
@@ -6,15 +6,15 @@
     <inertial>
       <origin
-        xyz="-0.0153035409571499 -0.000104495056790101 0.144451320818239"
-        rpy="0 0 0" />
-      <mass
-        value="8.36976133771814" />
-      <inertia
-        ixx="0.134439534189409"
-        ixy="0.000113435598147749"
-        ixz="-0.000259638829695405"
-        iyy="0.160334514687276"
-        iyz="7.17858064248926E-06"
-        izz="0.286274281412351" />
+        xyz="0.00298593644358607 -0.000268295172875241 0.154640959753498"
+        rpy="0 0 0" />
+      <mass
+        value="12.0012331336924" />
+      <inertia
+        ixx="0.35866059453322"
+        ixy="4.67770377513155E-08"
+        ixz="0.000423861580413772"
+        iyy="0.233823654906046"
+        iyz="4.66362844507336E-09"
+        izz="0.375131573810826" />
     </inertial>
     <visual>
@@ -51,37 +51,37 @@
     <inertial>
       <origin
-        xyz="1.29063426612674E-15 0.0290000000000001 -7.56339435525888E-16"
-        rpy="0 0 0" />
-      <mass
-        value="1.67636522822888" />
-      <inertia
-        ixx="0.00437925095774994"
-        ixy="9.37334798540553E-36"
-        ixz="-6.39017288398117E-36"
-        iyy="0.00781861981087289"
-        iyz="-1.19327077841116E-17"
-        izz="0.00437925095774994" />
-    </inertial>
-    <visual>
-      <origin
-        xyz="0 0 0"
-        rpy="0 0 0" />
-      <geometry>
-        <mesh
-          filename="package://rospital_description/meshes/WL_Link.STL" />
-      </geometry>
-      <material
-        name="">
-        <color
-          rgba="0.792156862745098 0.819607843137255 0.933333333333333 1" />
-      </material>
-    </visual>
-    <collision>
-      <origin
-        xyz="0 0 0"
-        rpy="0 0 0" />
-      <geometry>
-        <mesh
-          filename="package://rospital_description/meshes/WL_Link.STL" />
+        xyz="-8.64344718974191E-06 0.0228237946886783 7.57765177879927E-08"
+        rpy="0 0 0" />
+      <mass
+        value="0.778339693950675" />
+      <inertia
+        ixx="0.00165430356623842"
+        ixy="6.08982301451092E-09"
+        ixz="3.56600628105672E-11"
+        iyy="0.0030911762450513"
+        iyz="-2.8372582055542E-11"
+        izz="0.00165423410528579" />
+    </inertial>
+    <visual>
+      <origin
+        xyz="0 0 0"
+        rpy="0 0 0" />
+      <geometry>
+        <mesh
+          filename="package://rospital_description/meshes/wheel_left_link.STL" />
+      </geometry>
+      <material
+        name="">
+        <color
+          rgba="0.792156862745098 0.819607843137255 0.933333333333333 1" />
+      </material>
+    </visual>
+    <collision>
+      <origin
+        xyz="0 0 0"
+        rpy="0 0 0" />
+      <geometry>
+        <mesh
+          filename="package://rospital_description/meshes/wheel_left_link.STL" />
       </geometry>
     </collision>
@@ -91,6 +91,6 @@
     type="continuous">
     <origin
-      xyz="-0.00997450704782056 -0.165 0.0424413114931455"
-      rpy="0 0 3.14159265358979" />
+      xyz="0 0.161 0.0154413114931434"
+      rpy="0 0 0" />
     <parent
       link="base_link" />
@@ -98,5 +98,5 @@
       link="wheel_left_link" />
     <axis
-      xyz="0 -1 0" />
+      xyz="0 1 0" />
   </joint>
   <link
@@ -104,37 +104,37 @@
     <inertial>
       <origin
-        xyz="-1.0998146837693E-15 0.0290000000000001 -7.91033905045424E-16"
-        rpy="0 0 0" />
-      <mass
-        value="1.67636522822888" />
-      <inertia
-        ixx="0.00437925095774994"
-        ixy="2.48183918923532E-35"
-        ixz="1.97548076031495E-35"
-        iyy="0.00781861981087289"
-        iyz="-1.20253009911148E-17"
-        izz="0.00437925095774994" />
-    </inertial>
-    <visual>
-      <origin
-        xyz="0 0 0"
-        rpy="0 0 0" />
-      <geometry>
-        <mesh
-          filename="package://rospital_description/meshes/WR_Link.STL" />
-      </geometry>
-      <material
-        name="">
-        <color
-          rgba="0.792156862745098 0.819607843137255 0.933333333333333 1" />
-      </material>
-    </visual>
-    <collision>
-      <origin
-        xyz="0 0 0"
-        rpy="0 0 0" />
-      <geometry>
-        <mesh
-          filename="package://rospital_description/meshes/WR_Link.STL" />
+        xyz="8.64344718911542E-06 -0.0228237946886785 7.57765181002429E-08"
+        rpy="0 0 0" />
+      <mass
+        value="0.778339693950669" />
+      <inertia
+        ixx="0.00165430356623842"
+        ixy="6.08982301952646E-09"
+        ixz="-3.56600611496615E-11"
+        iyy="0.00309117624505131"
+        iyz="2.83725665326271E-11"
+        izz="0.0016542341052858" />
+    </inertial>
+    <visual>
+      <origin
+        xyz="0 0 0"
+        rpy="0 0 0" />
+      <geometry>
+        <mesh
+          filename="package://rospital_description/meshes/wheel_right_link.STL" />
+      </geometry>
+      <material
+        name="">
+        <color
+          rgba="0.792156862745098 0.819607843137255 0.933333333333333 1" />
+      </material>
+    </visual>
+    <collision>
+      <origin
+        xyz="0 0 0"
+        rpy="0 0 0" />
+      <geometry>
+        <mesh
+          filename="package://rospital_description/meshes/wheel_right_link.STL" />
       </geometry>
     </collision>
@@ -144,5 +144,5 @@
     type="continuous">
     <origin
-      xyz="-0.00998549295217773 0.165 0.0424413114931452"
+      xyz="0 -0.161 0.0154413114931451"
       rpy="0 0 0" />
     <parent
@@ -154,106 +154,106 @@
   </joint>
   <link
-    name="SF_link">
-    <inertial>
-      <origin
-        xyz="-0.000741617479152856 -0.000440542655304963 0.000304836017723242"
-        rpy="0 0 0" />
-      <mass
-        value="0.0226599458506464" />
-      <inertia
-        ixx="3.04243352925476E-06"
-        ixy="-1.06228231488976E-20"
-        ixz="-2.10390463354871E-11"
-        iyy="4.69226610526888E-06"
-        iyz="2.44129737654398E-21"
-        izz="3.04246223108001E-06" />
-    </inertial>
-    <visual>
-      <origin
-        xyz="0 0 0"
-        rpy="0 0 0" />
-      <geometry>
-        <mesh
-          filename="package://rospital_description/meshes/SF_Link.STL" />
-      </geometry>
-      <material
-        name="">
-        <color
-          rgba="0.792156862745098 0.819607843137255 0.933333333333333 1" />
-      </material>
-    </visual>
-    <collision>
-      <origin
-        xyz="0 0 0"
-        rpy="0 0 0" />
-      <geometry>
-        <mesh
-          filename="package://rospital_description/meshes/SF_Link.STL" />
-      </geometry>
-    </collision>
-  </link>
-  <joint
-    name="SF_joint"
+    name="caster_front_link">
+    <inertial>
+      <origin
+        xyz="0.000805650652548229 5.72729797615468E-17 -4.48165838715792E-06"
+        rpy="0 0 0" />
+      <mass
+        value="0.0386238363179237" />
+      <inertia
+        ixx="7.66294109641648E-06"
+        ixy="-1.82721726780336E-20"
+        ixz="2.42889623642253E-11"
+        iyy="1.29044379500025E-05"
+        iyz="-4.77133079419545E-24"
+        izz="7.66293122817673E-06" />
+    </inertial>
+    <visual>
+      <origin
+        xyz="0 0 0"
+        rpy="0 0 0" />
+      <geometry>
+        <mesh
+          filename="package://rospital_description/meshes/caster_front_link.STL" />
+      </geometry>
+      <material
+        name="">
+        <color
+          rgba="0.792156862745098 0.819607843137255 0.933333333333333 1" />
+      </material>
+    </visual>
+    <collision>
+      <origin
+        xyz="0 0 0"
+        rpy="0 0 0" />
+      <geometry>
+        <mesh
+          filename="package://rospital_description/meshes/caster_front_link.STL" />
+      </geometry>
+    </collision>
+  </link>
+  <joint
+    name="caster_front_joint"
     type="fixed">
     <origin
-      xyz="0.205921758347577 0 -0.0334694761074416"
-      rpy="0 0 0" />
-    <parent
-      link="base_link" />
-    <child
-      link="SF_link" />
+      xyz="0.229250238887004 -0.000124017376899337 -0.0431115511971616"
+      rpy="0 0 0" />
+    <parent
+      link="base_link" />
+    <child
+      link="caster_front_link" />
     <axis
       xyz="0 0 0" />
   </joint>
   <link
-    name="SB_link">
-    <inertial>
-      <origin
-        xyz="-0.000741617479152828 -0.000440542655306468 0.000304836017723242"
-        rpy="0 0 0" />
-      <mass
-        value="0.0226599458506464" />
-      <inertia
-        ixx="3.04243352925476E-06"
-        ixy="-1.06229858046925E-20"
-        ixz="-2.10390463355186E-11"
-        iyy="4.69226610526888E-06"
-        iyz="2.4415141565532E-21"
-        izz="3.04246223108001E-06" />
-    </inertial>
-    <visual>
-      <origin
-        xyz="0 0 0"
-        rpy="0 0 0" />
-      <geometry>
-        <mesh
-          filename="package://rospital_description/meshes/SB_Link.STL" />
-      </geometry>
-      <material
-        name="">
-        <color
-          rgba="0.792156862745098 0.819607843137255 0.933333333333333 1" />
-      </material>
-    </visual>
-    <collision>
-      <origin
-        xyz="0 0 0"
-        rpy="0 0 0" />
-      <geometry>
-        <mesh
-          filename="package://rospital_description/meshes/SB_Link.STL" />
-      </geometry>
-    </collision>
-  </link>
-  <joint
-    name="SB_joint"
+    name="caster_rear_link">
+    <inertial>
+      <origin
+        xyz="-0.000805650652548229 -6.01461155186334E-17 -4.48165838716486E-06"
+        rpy="0 0 0" />
+      <mass
+        value="0.0386238363179237" />
+      <inertia
+        ixx="7.66294109641648E-06"
+        ixy="-3.86943114962554E-20"
+        ixz="-2.42889623642257E-11"
+        iyy="1.29044379500025E-05"
+        iyz="-7.32910421549178E-20"
+        izz="7.66293122817673E-06" />
+    </inertial>
+    <visual>
+      <origin
+        xyz="0 0 0"
+        rpy="0 0 0" />
+      <geometry>
+        <mesh
+          filename="package://rospital_description/meshes/caster_rear_link.STL" />
+      </geometry>
+      <material
+        name="">
+        <color
+          rgba="0.792156862745098 0.819607843137255 0.933333333333333 1" />
+      </material>
+    </visual>
+    <collision>
+      <origin
+        xyz="0 0 0"
+        rpy="0 0 0" />
+      <geometry>
+        <mesh
+          filename="package://rospital_description/meshes/caster_rear_link.STL" />
+      </geometry>
+    </collision>
+  </link>
+  <joint
+    name="caster_rear_joint"
     type="fixed">
     <origin
-      xyz="-0.204078241652423 0 -0.0334694761074416"
-      rpy="0 0 0" />
-    <parent
-      link="base_link" />
-    <child
-      link="SB_link" />
+      xyz="-0.229157886818826 -0.000123712642857387 -0.0431115511971648"
+      rpy="0 0 0" />
+    <parent
+      link="base_link" />
+    <child
+      link="caster_rear_link" />
     <axis
       xyz="0 0 0" />
