Commit message: Update src packages

File: src/ rospital_description/urdf/rospital_gazebo.xacro (robot description, xacro)
@@ -18,6 +18,6 @@
   <gazebo reference="wheel_left_link">
     <material>Gazebo/Blue</material>
-    <mu1>1.0</mu1>
-    <mu2>1.0</mu2>
+    <mu1>1000000000000000.0</mu1>
+    <mu2>1000000000000000.0</mu2>
     <kp>1000000000000.0</kp>
     <kd>10.0</kd>
@@ -28,6 +28,6 @@
   <gazebo reference="wheel_right_link">
     <material>Gazebo/Blue</material>
-    <mu1>1.0</mu1>
-    <mu2>1.0</mu2>
+    <mu1>1000000000000000.0</mu1>
+    <mu2>1000000000000000.0</mu2>
     <kp>1000000000000.0</kp>
     <kd>10.0</kd>
@@ -37,5 +37,5 @@
   </gazebo>
   <!-- Caster Wheels -->
-  <gazebo reference="SB_link">
+  <gazebo reference="caster_rear_link">
     <material>Gazebo/FlatBlack</material>
     <mu1>0.1</mu1>
@@ -46,5 +46,5 @@
     <maxVel>1.0</maxVel>
   </gazebo>
-  <gazebo reference="SF_link">
+  <gazebo reference="caster_front_link">
     <material>Gazebo/FlatBlack</material>
     <mu1>0.1</mu1>
@@ -148,161 +148,161 @@
     </sensor>
   </gazebo>
-  <gazebo reference="F1_link">
-    <sensor name="F1" type="ray">
-      <always_on>true</always_on>
-      <visualize>true</visualize>
-      <update_rate>50</update_rate>
-      <ray>
-        <scan>
-          <horizontal>
-            <samples>5</samples>
-            <resolution>1.00000</resolution>
-            <min_angle>-0.14835</min_angle>
-            <max_angle>0.14835</max_angle>
-          </horizontal>
-        </scan>
-        <range>
-          <min>0.120000</min>
-          <max>4.0</max>
-          <resolution>0.015000</resolution>
-        </range>
-      </ray>
-      <plugin filename="libgazebo_ros_ray_sensor.so" name="f1_plugin">
-        <ros>
-          <remapping>~/out:=F1</remapping>
-        </ros>
-        <output_type>sensor_msgs/Range</output_type>
-        <frameName>F1_link</frameName>
-        <radiation_type>ultrasound</radiation_type>
-        <fov>0.2967</fov>
-      </plugin>
-    </sensor>
-  </gazebo>
-  <gazebo reference="F2_link">
-    <sensor name="F2" type="ray">
-      <always_on>true</always_on>
-      <visualize>true</visualize>
-      <update_rate>50</update_rate>
-      <ray>
-        <scan>
-          <horizontal>
-            <samples>5</samples>
-            <resolution>1.00000</resolution>
-            <min_angle>-0.14835</min_angle>
-            <max_angle>0.14835</max_angle>
-          </horizontal>
-        </scan>
-        <range>
-          <min>0.120000</min>
-          <max>4.0</max>
-          <resolution>0.015000</resolution>
-        </range>
-      </ray>
-      <plugin filename="libgazebo_ros_ray_sensor.so" name="f2_plugin">
-        <ros>
-          <remapping>~/out:=F2</remapping>
-        </ros>
-        <output_type>sensor_msgs/Range</output_type>
-        <frameName>F2_link</frameName>
-        <radiation_type>ultrasound</radiation_type>
-        <fov>0.2967</fov>
-      </plugin>
-    </sensor>
-  </gazebo>
-  <gazebo reference="L1_link">
-    <sensor name="L1" type="ray">
-      <always_on>true</always_on>
-      <visualize>true</visualize>
-      <update_rate>50</update_rate>
-      <ray>
-        <scan>
-          <horizontal>
-            <samples>5</samples>
-            <resolution>1.00000</resolution>
-            <min_angle>-0.14835</min_angle>
-            <max_angle>0.14835</max_angle>
-          </horizontal>
-        </scan>
-        <range>
-          <min>0.120000</min>
-          <max>4.0</max>
-          <resolution>0.015000</resolution>
-        </range>
-      </ray>
-      <plugin filename="libgazebo_ros_ray_sensor.so" name="l1_plugin">
-        <ros>
-          <remapping>~/out:=L1</remapping>
-        </ros>
-        <output_type>sensor_msgs/Range</output_type>
-        <frameName>L1_link</frameName>
-        <radiation_type>ultrasound</radiation_type>
-        <fov>0.2967</fov>
-      </plugin>
-    </sensor>
-  </gazebo>
-  <gazebo reference="L2_link">
-    <sensor name="L2" type="ray">
-      <always_on>true</always_on>
-      <visualize>true</visualize>
-      <update_rate>50</update_rate>
-      <ray>
-        <scan>
-          <horizontal>
-            <samples>5</samples>
-            <resolution>1.00000</resolution>
-            <min_angle>-0.14835</min_angle>
-            <max_angle>0.14835</max_angle>
-          </horizontal>
-        </scan>
-        <range>
-          <min>0.120000</min>
-          <max>4.0</max>
-          <resolution>0.015000</resolution>
-        </range>
-      </ray>
-      <plugin filename="libgazebo_ros_ray_sensor.so" name="l2_plugin">
-        <ros>
-          <remapping>~/out:=L2</remapping>
-        </ros>
-        <output_type>sensor_msgs/Range</output_type>
-        <frameName>L2_link</frameName>
-        <radiation_type>ultrasound</radiation_type>
-        <fov>0.2967</fov>
-      </plugin>
-    </sensor>
-  </gazebo>
-  <gazebo reference="R1_link">
-    <sensor name="R1" type="ray">
-      <always_on>true</always_on>
-      <visualize>true</visualize>
-      <update_rate>50</update_rate>
-      <ray>
-        <scan>
-          <horizontal>
-            <samples>5</samples>
-            <resolution>1.00000</resolution>
-            <min_angle>-0.14835</min_angle>
-            <max_angle>0.14835</max_angle>
-          </horizontal>
-        </scan>
-        <range>
-          <min>0.120000</min>
-          <max>4.0</max>
-          <resolution>0.015000</resolution>
-        </range>
-      </ray>
-      <plugin filename="libgazebo_ros_ray_sensor.so" name="r1_plugin">
-        <ros>
-          <remapping>~/out:=R1</remapping>
-        </ros>
-        <output_type>sensor_msgs/Range</output_type>
-        <frameName>R1_link</frameName>
-        <radiation_type>ultrasound</radiation_type>
-        <fov>0.2967</fov>
-      </plugin>
-    </sensor>
-  </gazebo>
-  <gazebo reference="R2_link">
-    <sensor name="R2" type="ray">
+  <gazebo reference="USB_link">
+    <sensor name="USB" type="ray">
+      <always_on>true</always_on>
+      <visualize>true</visualize>
+      <update_rate>50</update_rate>
+      <ray>
+        <scan>
+          <horizontal>
+            <samples>5</samples>
+            <resolution>1.00000</resolution>
+            <min_angle>-0.14835</min_angle>
+            <max_angle>0.14835</max_angle>
+          </horizontal>
+        </scan>
+        <range>
+          <min>0.120000</min>
+          <max>4.0</max>
+          <resolution>0.015000</resolution>
+        </range>
+      </ray>
+      <plugin filename="libgazebo_ros_ray_sensor.so" name="usb_plugin">
+        <ros>
+          <remapping>~/out:=ultrasound_1</remapping>
+        </ros>
+        <output_type>sensor_msgs/Range</output_type>
+        <frameName>USB_link</frameName>
+        <radiation_type>ultrasound</radiation_type>
+        <fov>0.2967</fov>
+      </plugin>
+    </sensor>
+  </gazebo>
+  <gazebo reference="USL1_link">
+    <sensor name="USL1" type="ray">
+      <always_on>true</always_on>
+      <visualize>true</visualize>
+      <update_rate>50</update_rate>
+      <ray>
+        <scan>
+          <horizontal>
+            <samples>5</samples>
+            <resolution>1.00000</resolution>
+            <min_angle>-0.14835</min_angle>
+            <max_angle>0.14835</max_angle>
+          </horizontal>
+        </scan>
+        <range>
+          <min>0.120000</min>
+          <max>4.0</max>
+          <resolution>0.015000</resolution>
+        </range>
+      </ray>
+      <plugin filename="libgazebo_ros_ray_sensor.so" name="usl1_plugin">
+        <ros>
+          <remapping>~/out:=ultrasound_2</remapping>
+        </ros>
+        <output_type>sensor_msgs/Range</output_type>
+        <frameName>USL1_link</frameName>
+        <radiation_type>ultrasound</radiation_type>
+        <fov>0.2967</fov>
+      </plugin>
+    </sensor>
+  </gazebo>
+  <gazebo reference="USL2_link">
+    <sensor name="USL2" type="ray">
+      <always_on>true</always_on>
+      <visualize>true</visualize>
+      <update_rate>50</update_rate>
+      <ray>
+        <scan>
+          <horizontal>
+            <samples>5</samples>
+            <resolution>1.00000</resolution>
+            <min_angle>-0.14835</min_angle>
+            <max_angle>0.14835</max_angle>
+          </horizontal>
+        </scan>
+        <range>
+          <min>0.120000</min>
+          <max>4.0</max>
+          <resolution>0.015000</resolution>
+        </range>
+      </ray>
+      <plugin filename="libgazebo_ros_ray_sensor.so" name="usl2_plugin">
+        <ros>
+          <remapping>~/out:=ultrasound_3</remapping>
+        </ros>
+        <output_type>sensor_msgs/Range</output_type>
+        <frameName>USL2_link</frameName>
+        <radiation_type>ultrasound</radiation_type>
+        <fov>0.2967</fov>
+      </plugin>
+    </sensor>
+  </gazebo>
+  <gazebo reference="USR1_link">
+    <sensor name="USR1" type="ray">
+      <always_on>true</always_on>
+      <visualize>true</visualize>
+      <update_rate>50</update_rate>
+      <ray>
+        <scan>
+          <horizontal>
+            <samples>5</samples>
+            <resolution>1.00000</resolution>
+            <min_angle>-0.14835</min_angle>
+            <max_angle>0.14835</max_angle>
+          </horizontal>
+        </scan>
+        <range>
+          <min>0.120000</min>
+          <max>4.0</max>
+          <resolution>0.015000</resolution>
+        </range>
+      </ray>
+      <plugin filename="libgazebo_ros_ray_sensor.so" name="usr1_plugin">
+        <ros>
+          <remapping>~/out:=ultrasound_4</remapping>
+        </ros>
+        <output_type>sensor_msgs/Range</output_type>
+        <frameName>USR1_link</frameName>
+        <radiation_type>ultrasound</radiation_type>
+        <fov>0.2967</fov>
+      </plugin>
+    </sensor>
+  </gazebo>
+  <gazebo reference="USR2_link">
+    <sensor name="USR2" type="ray">
+      <always_on>true</always_on>
+      <visualize>true</visualize>
+      <update_rate>50</update_rate>
+      <ray>
+        <scan>
+          <horizontal>
+            <samples>5</samples>
+            <resolution>1.00000</resolution>
+            <min_angle>-0.14835</min_angle>
+            <max_angle>0.14835</max_angle>
+          </horizontal>
+        </scan>
+        <range>
+          <min>0.120000</min>
+          <max>4.0</max>
+          <resolution>0.015000</resolution>
+        </range>
+      </ray>
+      <plugin filename="libgazebo_ros_ray_sensor.so" name="usr2_plugin">
+        <ros>
+          <remapping>~/out:=ultrasound_5</remapping>
+        </ros>
+        <output_type>sensor_msgs/Range</output_type>
+        <frameName>USR2_link</frameName>
+        <radiation_type>ultrasound</radiation_type>
+        <fov>0.2967</fov>
+      </plugin>
+    </sensor>
+  </gazebo>
+  <gazebo reference="USF_link">
+    <sensor name="USF" type="ray">
       <always_on>true</always_on>
       <visualize>true</visualize>
@@ -323,72 +323,10 @@
         </range>
       </ray>
-      <plugin filename="libgazebo_ros_ray_sensor.so" name="r2_plugin">
-        <ros>
-          <remapping>~/out:=R2</remapping>
-        </ros>
-        <output_type>sensor_msgs/Range</output_type>
-        <frameName>R2_link</frameName>
-        <radiation_type>ultrasound</radiation_type>
-        <fov>0.2967</fov>
-      </plugin>
-    </sensor>
-  </gazebo>
-  <gazebo reference="B1_link">
-    <sensor name="B1" type="ray">
-      <always_on>true</always_on>
-      <visualize>true</visualize>
-      <update_rate>50</update_rate>
-      <ray>
-        <scan>
-          <horizontal>
-            <samples>5</samples>
-            <resolution>1.00000</resolution>
-            <min_angle>-0.14835</min_angle>
-            <max_angle>0.14835</max_angle>
-          </horizontal>
-        </scan>
-        <range>
-          <min>0.120000</min>
-          <max>4.0</max>
-          <resolution>0.015000</resolution>
-        </range>
-      </ray>
-      <plugin filename="libgazebo_ros_ray_sensor.so" name="b1_plugin">
-        <ros>
-          <remapping>~/out:=B1</remapping>
-        </ros>
-        <output_type>sensor_msgs/Range</output_type>
-        <frameName>B1_link</frameName>
-        <radiation_type>ultrasound</radiation_type>
-        <fov>0.2967</fov>
-      </plugin>
-    </sensor>
-  </gazebo>
-  <gazebo reference="B2_link">
-    <sensor name="B2" type="ray">
-      <always_on>true</always_on>
-      <visualize>true</visualize>
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
File: src/ rospital_description/urdf/ultrasonic.xacro (robot description, xacro)
@@ -2,424 +2,318 @@
 <robot xmlns:xacro="http://ros.org/wiki/xacro">
   <link
-    name="R2_link">
-    <inertial>
-      <origin
-        xyz="-0.0025 2.77555756156289E-17 1.38777878078145E-17"
-        rpy="0 0 0" />
-      <mass
-        value="0.00495" />
-      <inertia
-        ixx="1.0349625E-06"
-        ixy="-5.81793843725135E-21"
-        ixz="-5.96110879390941E-22"
-        iyy="2.099625E-07"
-        iyz="4.31007979377368E-21"
-        izz="8.45625000000001E-07" />
-    </inertial>
-    <visual>
-      <origin
-        xyz="0 0 0"
-        rpy="0 0 0" />
-      <geometry>
-        <mesh
-          filename="package://rospital_description/meshes/SSR2_Link.STL" />
-      </geometry>
-      <material
-        name="">
-        <color
-          rgba="0.792156862745098 0.819607843137255 0.933333333333333 1" />
-      </material>
-    </visual>
-    <collision>
-      <origin
-        xyz="0 0 0"
-        rpy="0 0 0" />
-      <geometry>
-        <mesh
-          filename="package://rospital_description/meshes/SSR2_Link.STL" />
-      </geometry>
-    </collision>
-  </link>
-  <joint
-    name="R2_joint"
-    type="fixed">
-    <origin
-      xyz="-0.19111 0.2 0.053"
-      rpy="0 0 1.5708" />
-    <parent
-      link="base_link" />
-    <child
-      link="R2_link" />
-    <axis
-      xyz="0 0 0" />
-  </joint>
-  <link
-    name="R1_link">
-    <inertial>
-      <origin
-        xyz="-0.00249999999999997 0 6.93889390390723E-18"
-        rpy="0 0 0" />
-      <mass
-        value="0.00495" />
-      <inertia
-        ixx="1.0349625E-06"
-        ixy="-5.81793843725135E-21"
-        ixz="-5.96110879390941E-22"
-        iyy="2.099625E-07"
-        iyz="4.31007979377368E-21"
-        izz="8.45625000000001E-07" />
-    </inertial>
-    <visual>
-      <origin
-        xyz="0 0 0"
-        rpy="0 0 0" />
-      <geometry>
-        <mesh
-          filename="package://rospital_description/meshes/SSR1_Link.STL" />
-      </geometry>
-      <material
-        name="">
-        <color
-          rgba="0.792156862745098 0.819607843137255 0.933333333333333 1" />
-      </material>
-    </visual>
-    <collision>
-      <origin
-        xyz="0 0 0"
-        rpy="0 0 0" />
-      <geometry>
-        <mesh
-          filename="package://rospital_description/meshes/SSR1_Link.STL" />
-      </geometry>
-    </collision>
-  </link>
-  <joint
-    name="R1_joint"
-    type="fixed">
-    <origin
-      xyz="0.17111 0.2 0.053"
-      rpy="0 0 1.5708" />
-    <parent
-      link="base_link" />
-    <child
-      link="R1_link" />
-    <axis
-      xyz="0 0 0" />
-  </joint>
-  <link
-    name="L1_link">
-    <inertial>
-      <origin
-        xyz="-0.3975 0.000200000000764616 3.82339992999192E-13"
-        rpy="0 0 0" />
-      <mass
-        value="0.00495" />
-      <inertia
-        ixx="1.0349625E-06"
-        ixy="-5.81619484816385E-21"
-        ixz="-5.93312192183031E-22"
-        iyy="2.099625E-07"
-        iyz="4.36097619657057E-21"
-        izz="8.45625000000001E-07" />
-    </inertial>
-    <visual>
-      <origin
-        xyz="0 0 0"
-        rpy="0 0 0" />
-      <geometry>
-        <mesh
-          filename="package://rospital_description/meshes/SSL1_Link.STL" />
-      </geometry>
-      <material
-        name="">
-        <color
-          rgba="0.792156862745098 0.819607843137255 0.933333333333333 1" />
-      </material>
-    </visual>
-    <collision>
-      <origin
-        xyz="0 0 0"
-        rpy="0 0 0" />
-      <geometry>
-        <mesh
-          filename="package://rospital_description/meshes/SSL1_Link.STL" />
-      </geometry>
-    </collision>
-  </link>
-  <joint
-    name="L1_joint"
-    type="fixed">
-    <origin
-      xyz="0.17111 0.2 0.053"
-      rpy="0 0 1.5708" />
-    <parent
-      link="base_link" />
-    <child
-      link="L1_link" />
-    <axis
-      xyz="0 0 0" />
-  </joint>
-  <link
-    name="L2_link">
-    <inertial>
-      <origin
-        xyz="-0.3975 2.77555756156289E-15 1.39471767468535E-15"
-        rpy="0 0 0" />
-      <mass
-        value="0.00495" />
-      <inertia
-        ixx="1.0349625E-06"
-        ixy="-5.81619484816385E-21"
-        ixz="-5.93312192183032E-22"
-        iyy="2.099625E-07"
-        iyz="4.36097619657056E-21"
-        izz="8.45625000000001E-07" />
-    </inertial>
-    <visual>
-      <origin
-        xyz="0 0 0"
-        rpy="0 0 0" />
-      <geometry>
-        <mesh
-          filename="package://rospital_description/meshes/SSL2_Link.STL" />
-      </geometry>
-      <material
-        name="">
-        <color
-          rgba="0.792156862745098 0.819607843137255 0.933333333333333 1" />
-      </material>
-    </visual>
-    <collision>
-      <origin
-        xyz="0 0 0"
-        rpy="0 0 0" />
-      <geometry>
-        <mesh
-          filename="package://rospital_description/meshes/SSL2_Link.STL" />
-      </geometry>
-    </collision>
-  </link>
-  <joint
-    name="L2_joint"
-    type="fixed">
-    <origin
-      xyz="-0.19111 0.2 0.053"
-      rpy="0 0 1.5708" />
-    <parent
-      link="base_link" />
-    <child
-      link="L2_link" />
-    <axis
-      xyz="0 0 0" />
-  </joint>
-  <link
-    name="F1_link">
-    <inertial>
-      <origin
-        xyz="-0.00250000000000006 -5.55111512312578E-17 2.08166817117217E-17"
-        rpy="0 0 0" />
-      <mass
-        value="0.00495" />
-      <inertia
-        ixx="1.0349625E-06"
-        ixy="8.68146712826889E-21"
-        ixz="-1.41356690940057E-21"
-        iyy="2.099625E-07"
-        iyz="-2.18819838261876E-21"
-        izz="8.45625000000001E-07" />
-    </inertial>
-    <visual>
-      <origin
-        xyz="0 0 0"
-        rpy="0 0 0" />
-      <geometry>
-        <mesh
-          filename="package://rospital_description/meshes/SSF1_Link.STL" />
-      </geometry>
-      <material
-        name="">
-        <color
-          rgba="0.792156862745098 0.819607843137255 0.933333333333333 1" />
-      </material>
-    </visual>
-    <collision>
-      <origin
-        xyz="0 0 0"
-        rpy="0 0 0" />
-      <geometry>
-        <mesh
-          filename="package://rospital_description/meshes/SSF1_Link.STL" />
-      </geometry>
-    </collision>
-  </link>
-  <joint
-    name="F1_joint"
-    type="fixed">
-    <origin
-      xyz="0.24377 -0.1375 0.053"
+    name="USB_link">
+    <inertial>
+      <origin
+        xyz="0.00200485036829945 -6.30206112176707E-06 8.96260120698961E-05"
+        rpy="0 0 0" />
+      <mass
+        value="0.00351156143354723" />
+      <inertia
+        ixx="2.7228430247311E-07"
+        ixy="8.16918741171808E-14"
+        ixz="7.23554313169072E-12"
+        iyy="8.92094405089974E-08"
+        iyz="-2.49782595956578E-11"
+        izz="2.22970634830114E-07" />
+    </inertial>
+    <visual>
+      <origin
+        xyz="0 0 0"
+        rpy="0 0 0" />
+      <geometry>
+        <mesh
+          filename="package://rospital_description/meshes/USB_link.STL" />
+      </geometry>
+      <material
+        name="">
+        <color
+          rgba="0.752941176470588 0.752941176470588 0.752941176470588 1" />
+      </material>
+    </visual>
+    <collision>
+      <origin
+        xyz="0 0 0"
+        rpy="0 0 0" />
+      <geometry>
+        <mesh
+          filename="package://rospital_description/meshes/USB_link.STL" />
+      </geometry>
+    </collision>
+  </link>
+  <joint
+    name="USB_joint"
+    type="fixed">
+    <origin
+      xyz="-0.297247724970268 -0.000399525317885812 0.034797072321444"
+      rpy="0 0 -3.14" />
+    <parent
+      link="base_link" />
+    <child
+      link="USB_link" />
+    <axis
+      xyz="0 0 0" />
+  </joint>
+  <link
+    name="USL2_link">
+    <inertial>
+      <origin
+        xyz="0.00200465694765273 -2.85523787015851E-05 8.96260115198499E-05"
+        rpy="0 0 0" />
+      <mass
+        value="0.00351156143354724" />
+      <inertia
+        ixx="8.92094405089983E-08"
+        ixy="-8.169187091625E-14"
+        ixz="-2.49782595941744E-11"
+        iyy="2.7228430247311E-07"
+        iyz="-7.23554313158618E-12"
+        izz="2.22970634830115E-07" />
+    </inertial>
+    <visual>
+      <origin
+        xyz="0 0 0"
+        rpy="0 0 0" />
+      <geometry>
+        <mesh
+          filename="package://rospital_description/meshes/USL2_link.STL" />
+      </geometry>
+      <material
+        name="">
+        <color
+          rgba="0.752941176470588 0.752941176470588 0.752941176470588 1" />
+      </material>
+    </visual>
+    <collision>
+      <origin
+        xyz="0 0 0"
+        rpy="0 0 0" />
+      <geometry>
+        <mesh
+          filename="package://rospital_description/meshes/USL2_link.STL" />
+      </geometry>
+    </collision>
+  </link>
+  <joint
+    name="USL2_joint"
+    type="fixed">
+    <origin
+      xyz="-0.142436694016969 0.2 0.0347970723214464"
+      rpy="0 0 1.5707963267949" />
+    <parent
+      link="base_link" />
+    <child
+      link="USL2_link" />
+    <axis
+      xyz="0 0 0" />
+  </joint>
+  <link
+    name="USL1_link">
+    <inertial>
+      <origin
+        xyz="0.00200465694765256 -2.85523787028064E-05 8.96260115198569E-05"
+        rpy="0 0 0" />
+      <mass
+        value="0.00351156143354724" />
+      <inertia
+        ixx="8.92094405089983E-08"
+        ixy="-8.16918709175315E-14"
+        ixz="-2.49782595960476E-11"
+        iyy="2.7228430247311E-07"
+        iyz="-7.23554313158602E-12"
+        izz="2.22970634830115E-07" />
+    </inertial>
+    <visual>
+      <origin
+        xyz="0 0 0"
+        rpy="0 0 0" />
+      <geometry>
+        <mesh
+          filename="package://rospital_description/meshes/USL1_link.STL" />
+      </geometry>
+      <material
+        name="">
+        <color
+          rgba="0.752941176470588 0.752941176470588 0.752941176470588 1" />
+      </material>
+    </visual>
+    <collision>
+      <origin
+        xyz="0 0 0"
+        rpy="0 0 0" />
+      <geometry>
+        <mesh
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