Commit message: Cap nhat code moi nhat

File: src/ rospital_description/urdf/rospital.urdf.xacro (robot description, xacro)
@@ -8,3 +8,5 @@
     <xacro:include filename="imu.xacro"/>
     <xacro:include filename="ultrasonic.xacro"/>
+    <xacro:include filename="dual_arm.xacro"/>
+    <xacro:include filename="intel_rgbd_cam_d435.urdf.xacro" />
 </robot>

File: src/ rospital_description/urdf/rospital_gazebo.xacro (robot description, xacro)
@@ -1,18 +1,4 @@
 <?xml version="1.0"?>
 <robot name="rospital" xmlns:xacro="http://ros.org/wiki/xacro">
-  <transmission name="wheel_right_transmission">
-    <plugin>transmission_interface/SimpleTransmission</plugin>
-    <actuator name="wheel_right_motor" role="actuator_right"/>
-    <joint name="wheel_right_joint"    role="joint_right">
-      <mechanical_reduction>1.0</mechanical_reduction>
-    </joint>
-  </transmission>
-  <transmission name="wheel_left_transmission">
-    <plugin>transmission_interface/SimpleTransmission</plugin>
-    <actuator name="wheel_left_motor" role="actuator_left"/>
-    <joint name="wheel_left_joint"    role="joint_left">
-      <mechanical_reduction>1.0</mechanical_reduction>
-    </joint>
-  </transmission>
   <!-- Wheels -->
   <gazebo reference="wheel_left_link">

File: src/ rospital_description/urdf/rospital_ros2_control.xacro (robot description, xacro)
@@ -1,24 +1,4 @@
 <?xml version="1.0"?>
 <robot xmlns:xacro="http://www.ros.org/wiki/xacro" name="rospital">
-    <transmission name="right_wheel_trans">
-        <type>transmission_interface/SimpleTransmission</type>
-        <joint name="wheel_right_joint">
-            <hardwareInterface>hardware_interface::HW_IF_VELOCITY</hardwareInterface>
-        </joint>
-        <actuator name="right_wheel_motor">
-            <hardwareInterface>hardware_interface::HW_IF_VELOCITY</hardwareInterface>
-            <mechanicalReduction>1</mechanicalReduction>
-        </actuator>
-    </transmission>
-    <transmission name="left_wheel_trans">
-        <type>transmission_interface/SimpleTransmission</type>
-        <joint name="wheel_left_joint">
-            <hardwareInterface>hardware_interface::HW_IF_VELOCITY</hardwareInterface>
-        </joint>
-        <actuator name="left_wheel_motor">
-            <hardwareInterface>hardware_interface::HW_IF_VELOCITY</hardwareInterface>
-            <mechanicalReduction>1</mechanicalReduction>
-        </actuator>
-    </transmission>
     <ros2_control name="RobotSystem" type="system">
         <!-- ros2_control Gazebo -->
@@ -51,4 +31,54 @@
             <state_interface name="velocity" />
         </joint>
+        <joint name="left_shoulder_joint">
+            <command_interface name="position"/>
+            <state_interface name="position"/>
+            <state_interface name="velocity"/>
+        </joint>
+        <joint name="left_elbow_joint">
+            <command_interface name="position"/>
+            <state_interface name="position"/>
+            <state_interface name="velocity"/>
+        </joint>
+        <joint name="left_wrist_joint">
+            <command_interface name="position"/>
+            <state_interface name="position"/>
+            <state_interface name="velocity"/>
+        </joint>
+        <joint name="left_left_finger_joint">
+            <command_interface name="position"/>
+            <state_interface name="position"/>
+            <state_interface name="velocity"/>
+        </joint>
+        <joint name="left_right_finger_joint">
+            <command_interface name="position"/>
+            <state_interface name="position"/>
+            <state_interface name="velocity"/>
+        </joint>
+        <joint name="right_shoulder_joint">
+            <command_interface name="position"/>
+            <state_interface name="position"/>
+            <state_interface name="velocity"/>
+        </joint>
+        <joint name="right_elbow_joint">
+            <command_interface name="position"/>
+            <state_interface name="position"/>
+            <state_interface name="velocity"/>
+        </joint>
+        <joint name="right_wrist_joint">
+            <command_interface name="position"/>
+            <state_interface name="position"/>
+            <state_interface name="velocity"/>
+        </joint>
+        <joint name="right_left_finger_joint">
+            <command_interface name="position"/>
+            <state_interface name="position"/>
+            <state_interface name="velocity"/>
+        </joint>
+        <joint name="right_right_finger_joint">
+            <command_interface name="position"/>
+            <state_interface name="position"/>
+            <state_interface name="velocity"/>
+        </joint>
     </ros2_control>
 </robot>
